Commit message: ROS Braccio Arm

File: urdf/braccio.urdf (robot description, URDF)
Before this commit: robot braccio_arm, 9 links, 8 joints
Links:
- link gripper_base: geometry collision mesh filename=package://ros_braccio_arm/meshes/gripper_base.stl; visual mesh filename=package://ros_braccio_arm/meshes/gripper_base.stl
- link gripper_fix: geometry collision mesh filename=package://ros_braccio_arm/meshes/gripper_fix.stl; visual mesh filename=package://ros_braccio_arm/meshes/gripper_fix.stl
- link gripper_movable: geometry collision mesh filename=package://ros_braccio_arm/meshes/gripper_movable.stl; visual mesh filename=package://ros_braccio_arm/meshes/gripper_movable.stl
- link link1: geometry collision mesh filename=package://ros_braccio_arm/meshes/base.stl; visual mesh filename=package://ros_braccio_arm/meshes/base.stl
- link link2: geometry collision mesh filename=package://ros_braccio_arm/meshes/shoulder.stl; visual mesh filename=package://ros_braccio_arm/meshes/shoulder.stl
- link link3: geometry collision mesh filename=package://ros_braccio_arm/meshes/elbow.stl; visual mesh filename=package://ros_braccio_arm/meshes/elbow.stl
- link link4: geometry collision mesh filename=package://ros_braccio_arm/meshes/wrist_pitch.stl; visual mesh filename=package://ros_braccio_arm/meshes/wrist_pitch.stl
- link link5: geometry collision mesh filename=package://ros_braccio_arm/meshes/wrist_roll.stl; visual mesh filename=package://ros_braccio_arm/meshes/wrist_roll.stl
